File: hardware/epaper-breakout/epaper-breakout.sch (KiCad schematic (older format))
At the start: 68 parts, among them J1 XF2M-3315-1A, J2 C10418, J3 Conn_02x06_Counter_Clockwise, J4 ED060SC4, Q1 IRLML6402, U1 MCP1700-3302E_SOT23, U2 LT1945, U3 LT1945, U5 ESP32-WROVER, U6 CH330N, U7 LM358, U8 74HC4094-normal, U9 MCP9700AT-ETT

Commit message: update production files
Parts:
- L1, L2, L3, L4: LCSC (none) -> C326331
Changed lines of the file:
@@
 F 2 "Inductor_SMD:L_6.3x6.3_H3" H 2100 1150 50  0001 C CNN
 F 3 "~" H 2100 1150 50  0001 C CNN
+F 4 "C326331" V 2100 1150 50  0001 C CNN "LCSC"
 	1    2100 1150
 	0    1    1    0
@@
 F 2 "Inductor_SMD:L_6.3x6.3_H3" H 2100 2850 50  0001 C CNN
 F 3 "~" H 2100 2850 50  0001 C CNN
+F 4 "C326331" V 2100 2850 50  0001 C CNN "LCSC"
 	1    2100 2850
 	0    1    1    0
@@
 F 2 "Inductor_SMD:L_6.3x6.3_H3" H 9300 5750 50  0001 C CNN
 F 3 "~" H 9300 5750 50  0001 C CNN
+F 4 "C326331" V 9300 5750 50  0001 C CNN "LCSC"
 	1    9300 5750
 	0    1    1    0
@@
 F 2 "Inductor_SMD:L_6.3x6.3_H3" H 9300 7450 50  0001 C CNN
 F 3 "~" H 9300 7450 50  0001 C CNN
+F 4 "C326331" V 9300 7450 50  0001 C CNN "LCSC"
 	1    9300 7450
 	0    1    1    0
