File: hardware/ES108FC1_Connector/ES108FC1_Connector.kicad_sch (KiCad schematic)
At the start: 2 parts

Commit message: generate order files
Parts:
- added J1: Conn_02x03_Odd_Even, Connector_PinHeader_2.54mm:PinHeader_2x03_P2.54mm_Vertical, symbol Connector_Generic:Conn_02x03_Odd_Even
- J2: renamed from J?; footprint (none) -> epaper-breakout:ES108FC1; LCSC (none) -> C2880696
- U1: renamed from U?; footprint (none) -> epaper-breakout:Hirose_FH12-40S-0.5SH_mirrored; symbol epdiy:ED078KH6 -> epdiy:ED078KH6_REV; LCSC (none) -> C202114
Connections:
- net VGL: now reaches J2.1 (VGL), U1.1 (VGL)
- net VCOM: now reaches J2.7 (VCOM), U1.10 (VCOM)
- net VDD: now reaches J2.8 (VDD), U1.11 (VDD)
- net VDD: now also J2.3 (VDD), U1.5 (VDD)
- net GND: now reaches J2.9 (VSS), U1.12 (VSS), U1.9 (VSS)
- net GND: now also J2.27 (VSS), J2.39 (VSS), J2.40 (VSS), J2.45 (VSS), U1.22 (VSS), J1.2 (Pin_2)
- net XCL: now reaches J2.10 (XCL), U1.13 (XCL)
- net D0: now reaches U1.14 (D0)
- net D0: now also J2.11 (D0)
- net D1: now reaches U1.15 (D1)
- net D1: now also J2.13 (D1)
- net D2: now reaches U1.16 (D2)
- net D2: now also J2.15 (D2)
- net D3: now reaches U1.17 (D3)
- net D3: now also J2.17 (D3)
- net D4: now reaches U1.18 (D4)
- net D4: now also J2.19 (D4)
- net D5: now reaches U1.19 (D5)
- net D5: now also J2.21 (D5)
- net D6: now reaches U1.20 (D6)
- net D6: now also J2.23 (D6)
- net D7: now reaches U1.21 (D7)
- net D7: now also J2.25 (D7)
- net D8: now reaches U1.23 (D8)
- net D8: now also J2.12 (D8)
- net D9: now reaches U1.24 (D9)
- net D9: now also J2.14 (D9)
- net D10: now reaches U1.25 (D10)
- net D10: now also J2.16 (D10)
- net D11: now reaches U1.26 (D11)
- net D11: now also J2.18 (D11)
- net D12: now reaches U1.27 (D12)
- net D12: now also J2.20 (D12)
- net D13: now reaches U1.28 (D13)
- net D13: now also J2.22 (D13)
- net D14: now reaches U1.29 (D14)
- net D14: now also J2.24 (D14)
- net VGH: now reaches J2.2 (VGH), U1.3 (VGH)
- net D15: now reaches U1.30 (D15)
- net D15: now also J2.26 (D15)
- net XSTL: now reaches U1.31 (XSTL)
- net XSTL: now also J2.28 (XSTL)
- net XLE: now reaches U1.32 (XLE)
- net XLE: now also J2.29 (XLE)
- net XOE: now reaches U1.33 (XOE)
- net XOE: now also J2.30 (XOE)
- net TEST: now reaches U1.34 (TEST)
- net TEST: now also J2.31 (XON)
- net VPOS: now reaches U1.36 (VPOS)
- net VPOS: now also J2.32 (VPOS)
- net VNEG: now reaches U1.38 (VNEG)
- net VNEG: now also J2.33 (VNEG)
- net BRD: now reaches U1.40 (BORDER)
- net BRD: now also J2.34 (Border)
- net MODE: now reaches J2.4 (MODE), U1.6 (Mode)
- net CKV: now reaches J2.5 (CKV), U1.7 (CKV)
- net SPV: now reaches J2.6 (SPV), U1.8 (SPV)
- net SPI_VDD: now reaches J2.46 (VDD2)
- net SPI_VDD: now also J1.1 (Pin_1)
- net SPI_SCL: now reaches J2.47 (SPI_SCL)
- net SPI_SCL: now also J1.4 (Pin_4)
- net SPI_NCS: now reaches J2.48 (SPI_NCS)
- net SPI_NCS: now also J1.3 (Pin_3)
- net SPI_SDI: now reaches J2.49 (SPI_SDI)
- net SPI_SDI: now also J1.6 (Pin_6)
- net SPI_SDO: now reaches J2.50 (SPI_SDO)
- net SPI_SDO: now also J1.5 (Pin_5)
Other:
- moved on the sheet: J2
