File: hardware/epdiy-v7/epaper-breakout.kicad_sch (KiCad schematic)
At the start: 116 parts, among them J1 USB_C_Receptacle_USB2.0, J2 EXTENSION_HEADER, J3 ESP_HEADER, J4 XF2M-3315-1A, J5 CONN_BAT, J6 8BIT_HEADER, Q1 AO3401A, Q3 MMBT3904, Q4 MMBT3904, U1 RT9080-33GJ5, U10 ED060XC5, U11 TP4056, U2 PCA9535PW, U3 TPS651851RSLR, U4 USBLC6-2P6, U5 XC6206PxxxMR, U6 ED078KH6, U7 PCF8563T, U8 ESP32-S3-WROOM-1, U9 CH340C, Y1 32.768K

Commit message: v7 signal connections
Parts:
- removed J3: ESP_HEADER, Connector_PinHeader_2.54mm:PinHeader_1x13_P2.54mm_Vertical, symbol Connector:Conn_01x13_Female
- added J3: USB_HDR, Connector_PinHeader_2.54mm:PinHeader_1x02_P2.54mm_Vertical, symbol Connector:Conn_01x02_Female
- added J7: ESP_HDR, Connector_PinHeader_2.54mm:PinHeader_1x12_P2.54mm_Vertical, symbol Connector:Conn_01x12_Female
- J6: footprint (none) -> Connector_PinHeader_2.54mm:PinHeader_1x10_P2.54mm_Vertical
- U1: footprint TSOT-23-5_RIT -> Package_TO_SOT_SMD:TSOT-23-5
- U5: footprint Package_TO_SOT_SMD:SOT-23 -> Package_TO_SOT_SMD:SOT-23-3
Connections:
- net IO0 is gone; now on net EP_STV: Q4.3 (C), R15.1, U8.27 (GPIO0/BOOT)
- net 3.3V: now also J7.2 (Pin_2)
- net EP_STV: no longer U8.15 (GPIO3/TOUCH3/ADC1_CH2)
- net ESP_USB+: now also J3.2 (Pin_2)
- net ESP_USB-: now also J3.1 (Pin_1)
- net GND: now also J7.12 (Pin_12)
- net GPIO_1: now also JP1.1 (A), J7.3 (Pin_3); no longer JP2.2 (B)
- net GPIO_2: now also JP2.2 (B), J7.4 (Pin_4); no longer JP1.1 (A)
- net GPIO_35: now also J7.10 (Pin_10)
- net GPIO_36: now also J7.9 (Pin_9)
- net GPIO_37: now also J7.8 (Pin_8)
- net GPIO_45: now also J7.7 (Pin_7)
- net GPIO_46: now also J7.6 (Pin_6)
- net RTC_CLK: now also J7.11 (Pin_11)
- net VIN: now also J7.1 (Pin_1)
- new net GPIO_3: J7.5 (Pin_5), U8.15 (GPIO3/TOUCH3/ADC1_CH2)
Other:
- moved on the sheet: JP2, R32, R4, R6

Commit message: generate order files
Parts:
- C19: LCSC C19702 -> C15850
- C21, C41: LCSC (none) -> C1792
- C29: LCSC C49678 -> C49678
- J1: LCSC (none) -> C165948
- J4: LCSC (none) -> C231420
- Q1: LCSC (none) -> C15127
- R2, R7: LCSC (none) -> C23186
- R5: LCSC (none) -> C21189
- U1: LCSC (none) -> C841192
- U10: LCSC (none) -> C528053
- U4: LCSC (none) -> C2827693
- U5: LCSC (none) -> C5446
- U6: LCSC (none) -> C202114
- U7: LCSC (none) -> C7440
- U8: LCSC (none) -> C2913202
- U9: LCSC (none) -> C84681
Changed lines of the file:
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@@
       (effects (font (size 1.27 1.27)) hide)
     )
-    (property "LCSC" " C49678" (id 4) (at 139.7 205.74 0)
+    (property "LCSC" "C49678" (id 4) (at 139.7 205.74 0)
       (effects (font (size 1.27 1.27)) hide)
     )
@@
       (effects (font (size 1.27 1.27)) hide)
     )
-    (property "LCSC" "C19702" (id 4) (at 167.64 254 0)
+    (property "LCSC" "C15850" (id 4) (at 167.64 254 0)
       (effects (font (size 1.27 1.27)) hide)
     )
@@
       (effects (font (size 1.27 1.27)) hide)
     )
-    (property "LCSC" "" (id 4) (at 308.61 205.74 0)
+    (property "LCSC" "C21189" (id 4) (at 308.61 205.74 0)
       (effects (font (size 1.27 1.27)) hide)
     )
@@
       (effects (font (size 1.524 1.524)))
     )
+    (property "LCSC" "C841192" (id 4) (at 32.385 102.87 0)
+      (effects (font (size 1.27 1.27)) hide)
+    )
     (pin "1")
     (pin "2")
@@
       (effects (font (size 1.27 1.27)) hide)
     )
+    (property "LCSC" "C2913202" (id 4) (at 267.97 58.42 0)
+      (effects (font (size 1.27 1.27)) hide)
+    )
     (pin "1")
     (pin "10")
@@
       (effects (font (size 1.524 1.524)))
     )
+    (property "LCSC" "C231420" (id 4) (at 203.2 168.91 0)
+      (effects (font (size 1.27 1.27)) hide)
+    )
     (pin "1")
     (pin "10")
@@
       (effects (font (size 1.27 1.27)) hide)
     )
+    (property "LCSC" "C202114" (id 4) (at 379.73 29.21 0)
+      (effects (font (size 1.27 1.27)) hide)
+    )
     (pin "1")
     (pin "10")
@@
       (effects (font (size 1.27 1.27)) hide)
     )
+    (property "LCSC" "C84681" (id 4) (at 142.24 39.37 0)
+      (effects (font (size 1.27 1.27)) hide)
+    )
     (pin "1")
     (pin "10")
@@
       (effects (font (size 1.27 1.27)) hide)
     )
+    (property "LCSC" "C528053" (id 4) (at 264.16 208.28 0)
+      (effects (font (size 1.27 1.27)) hide)
+    )
     (pin "1")
     (pin "10")
@@
       (effects (font (size 1.27 1.27)) hide)
     )
+    (property "LCSC" "C165948" (id 4) (at 33.02 43.18 0)
+      (effects (font (size 1.27 1.27)) hide)
+    )
     (pin "A1")
     (pin "A12")
@@
       (effects (font (size 1.27 1.27)) hide)
     )
+    (property "LCSC" "C2827693" (id 4) (at 59.69 72.39 0)
+      (effects (font (size 1.27 1.27)) hide)
+    )
     (pin "1")
     (pin "2")
@@
       (effects (font (size 1.27 1.27)) hide)
     )
-    (property "LCSC" "" (id 4) (at 74.93 40.64 0)
+    (property "LCSC" "C23186" (id 4) (at 74.93 40.64 0)
       (effects (font (size 1.27 1.27)) hide)
     )
@@
       (effects (font (size 1.27 1.27)) hide)
     )
+    (property "LCSC" "C7440" (id 4) (at 256.54 110.49 0)
+      (effects (font (size 1.27 1.27)) hide)
+    )
     (pin "1")
     (pin "2")
@@
       (effects (font (size 1.27 1.27)) hide)
     )
+    (property "LCSC" "C5446" (id 4) (at 107.95 46.99 0)
+      (effects (font (size 1.27 1.27)) hide)
+    )
     (pin "1")
     (pin "2")
@@
       (effects (font (size 1.27 1.27)) hide)
     )
-    (property "LCSC" "" (id 4) (at 67.31 40.64 0)
+    (property "LCSC" "C23186" (id 4) (at 67.31 40.64 0)
       (effects (font (size 1.27 1.27)) hide)
     )
@@
       (effects (font (size 1.27 1.27)) hide)
     )
+    (property "LCSC" "C1792" (id 4) (at 231.775 115.57 0)
+      (effects (font (size 1.27 1.27)) hide)
+    )
     (pin "1")
     (pin "2")
@@
       (effects (font (size 1.27 1.27)) (justify left) hide)
     )
+    (property "LCSC" "C15127" (id 4) (at 52.07 130.81 0)
+      (effects (font (size 1.27 1.27)) hide)
+    )
     (pin "1")
     (pin "2")
@@
       (effects (font (size 1.27 1.27)) hide)
     )
+    (property "LCSC" "C1792" (id 4) (at 231.14 105.41 0)
+      (effects (font (size 1.27 1.27)) hide)
+    )
